File: keyboard.kicad_sch (KiCad schematic)
At the start: 20 parts, among them SW1 SW_Push, U1 ATmega32U4-A, Y1 16MHz

Commit message: pcb schematic
Parts:
- MX1, MX2: footprint MX_Alps_Hybrid:MX-1U-NoLED -> MX_Alps_Hybrid:MX-1U
Changed lines of the file:
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@@
       (effects (font (size 0.508 0.508)))
     )
-    (property "Footprint" "MX_Alps_Hybrid:MX-1U-NoLED" (id 2) (at 200.025 120.015 0)
+    (property "Footprint" "MX_Alps_Hybrid:MX-1U" (id 2) (at 200.025 120.015 0)
       (effects (font (size 1.524 1.524)) hide)
     )
@@
       (effects (font (size 0.508 0.508)))
     )
-    (property "Footprint" "MX_Alps_Hybrid:MX-1U-NoLED" (id 2) (at 184.785 120.015 0)
+    (property "Footprint" "MX_Alps_Hybrid:MX-1U" (id 2) (at 184.785 120.015 0)
       (effects (font (size 1.524 1.524)) hide)
     )
@@
     )
     (path "/c737769b-166a-4ea4-8d01-fd7d7d15ed2b"
-      (reference "MX1") (unit 1) (value "MX-NoLED") (footprint "MX_Alps_Hybrid:MX-1U-NoLED")
+      (reference "MX1") (unit 1) (value "MX-NoLED") (footprint "MX_Alps_Hybrid:MX-1U")
     )
     (path "/16d21747-c2b1-4e12-9fda-e6b266cbb054"
-      (reference "MX2") (unit 1) (value "MX-NoLED") (footprint "MX_Alps_Hybrid:MX-1U-NoLED")
+      (reference "MX2") (unit 1) (value "MX-NoLED") (footprint "MX_Alps_Hybrid:MX-1U")
     )
     (path "/7cefd24c-42cf-4fe8-bdf0-77759279f9da"
