File: keyboard.kicad_pcb (KiCad board)
At the start: 2 copper layers, 20 parts, among them SW1 SW_Push, U1 ATmega32U4-A, Y1 16MHz

Commit message: PCB Schematic
Parts:
- C1, C2, C3, C4, C5, C6, C7, D1, D2, R1, R2, R3, SW1, U1, Y1: moved to B.Cu
- moved D2 127.5 mm to (231.8, 69.8), turned to 90 degrees
- moved MX2 108.1 mm to (223.8, 69.8)
- moved MX1 69.3 mm to (204.8, 69.8)
- moved USB1 68.6 mm to (166.7, 58.7), turned to -90 degrees
- moved C6 67.5 mm to (189.7, 86.5), turned to 180 degrees
- moved D1 65.9 mm to (212.7, 69.8), turned to 90 degrees
- moved C4 64.9 mm to (176.2, 69.8), turned to 90 degrees
- moved R4 63.4 mm to (194.5, 82.5), turned to -90 degrees
- moved Y1 62.7 mm to (184.9, 66.7), turned to 180 degrees
- moved C2 61.4 mm to (181.0, 66.7), turned to -90 degrees
- moved C3 61.4 mm to (175.4, 77.8), turned to 180 degrees
- moved F1 56.0 mm to (161.9, 74.6), turned to 90 degrees
- moved R1 55.3 mm to (173.0, 69.8), turned to 90 degrees
- moved C5 48.3 mm to (193.7, 73.8), turned to 90 degrees
- moved C7 46.8 mm to (180.2, 86.5)
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Other:
- board outline added: 74.7 x 31.8 mm
